File: hardware/electronics/gps-lte.kicad_sch (KiCad schematic)
At the start: 62 parts, among them J11 U.FL-R-SMT-1(10), U10 AD8541ARTZ, U11 TXS0102DQER, U12 BGA725L6E6327FTSA1, U13 B39162B9416K610

Commit message: v5_update
Parts:
- ANT1: symbol Flatburn_V4_sym_library:LTE/GNSS/BT - 400-8000 MHz - NN03-310 -> FAE-ANT:LTE/GNSS/BT - 400-8000 MHz - NN03-310
- ANT2: symbol Flatburn_V4_sym_library:GNSS - 824-82000 MHz - NN02-224 -> FAE-ANT:GNSS - 824-82000 MHz - NN02-224
- C106: symbol Flatburn_V4_sym_library:CS-C-0402-1.6p/50V -> FAE-CAP:CS-C-0402-1.6p/50V
- C107: symbol Flatburn_V4_sym_library:CS-C-0402-0.4p/50V -> FAE-CAP:CS-C-0402-0.4p/50V
- C108: symbol Flatburn_V4_sym_library:CS-C-0402-0.5p/50V -> FAE-CAP:CS-C-0402-0.5p/50V
- C109: symbol Flatburn_V4_sym_library:CS-C-0402-0.3p/50V -> FAE-CAP:CS-C-0402-0.3p/50V
- C110, C111, C112, C113, C117, C118, C120: symbol Flatburn_V4_sym_library:CS-C-0402-100n/50V-10% -> FAE-CAP:CS-C-0402-100n/50V-10%
- C114: symbol Flatburn_V4_sym_library:CS-C-0402-1n/50V-10% -> FAE-CAP:CS-C-0402-1n/50V-10%
- C115: symbol Flatburn_V4_sym_library:SUPERCAP-EL-10.7x8.5-470mF/3.5V - FCS0V474ZFTBR24 -> FAE-CAP:SUPERCAP-EL-10.7x8.5-470mF/3.5V - FCS0V474ZFTBR24
- C116: symbol Flatburn_V4_sym_library:CS-C-0603-1u/25V-10% -> FAE-CAP:CS-C-0603-1u/25V-10%
- C119: symbol Flatburn_V4_sym_library:CS-C-0603-10u/10V-10% -> FAE-CAP:CS-C-0603-10u/10V-10%
- C121: symbol Flatburn_V4_sym_library:CS-C-0402-1u/16V-10% -> FAE-CAP:CS-C-0402-1u/16V-10%
- CABLE1: symbol Flatburn_V4_sym_library:U.FL -> FAE-CABLE:U.FL
- DS1: symbol Flatburn_V4_sym_library:SCHOTTKY - 30V/0.2A - BAT54J -> FAE-DIODES:SCHOTTKY - 30V/0.2A - BAT54J
- J11: symbol Flatburn_V4_sym_library:RF/COAX - U.FL-R-SMT-1(10) -> FAE-CONN:RF/COAX - U.FL-R-SMT-1(10)
- L10: symbol Flatburn_V4_sym_library:L RF - 15nH/1.4A - LQW18AN15NG80D -> FAE-IND:L RF - 15nH/1.4A - LQW18AN15NG80D
- L11: symbol Flatburn_V4_sym_library:L RF - 9.9nH/1.6A - LQW18AN9N9G80D -> FAE-IND:L RF - 9.9nH/1.6A - LQW18AN9N9G80D
- L12: symbol Flatburn_V4_sym_library:L RF - 10nH/1.6A - LQW18AN10NG80D -> FAE-IND:L RF - 10nH/1.6A - LQW18AN10NG80D
- L13: symbol Flatburn_V4_sym_library:L RF - 7.5nH/570mA - LQW15AN7N5H00D -> FAE-IND:L RF - 7.5nH/570mA - LQW15AN7N5H00D
- L14: symbol Flatburn_V4_sym_library:L RF - 7.1nH/1.42A - LQW15AN7N1G80D -> FAE-IND:L RF - 7.1nH/1.42A - LQW15AN7N1G80D
- L15: symbol Flatburn_V4_sym_library:L RF - 4.6nH/1.45A - LQW15AN4N6G80D -> FAE-IND:L RF - 4.6nH/1.45A - LQW15AN4N6G80D
- L8: symbol Flatburn_V4_sym_library:L RF - 1.3nH/3.15A - LQW15AN1N3C80D -> FAE-IND:L RF - 1.3nH/3.15A - LQW15AN1N3C80D
- L9: symbol Flatburn_V4_sym_library:L RF - 2.3nH/2.53A - LQW15AN2N3G80D -> FAE-IND:L RF - 2.3nH/2.53A - LQW15AN2N3G80D
- MOD1: symbol Flatburn_V4_sym_library:GPS/GNSS - NEO-M8U-06B -> FAE-MOD:GPS/GNSS - NEO-M8U-06B
- R145: symbol Flatburn_V4_sym_library:RS-0402-4K7 1/16W 1% -> FAE-RES:RS-0402-4K7 1/16W 1%
- R146, R148, R149, R165, R166, R167: symbol Flatburn_V4_sym_library:RS-0402-0R 100mW 0.1% -> FAE-RES:RS-0402-0R 100mW 0.1%
- R147, R153, R154: symbol Flatburn_V4_sym_library:RS-0402-0R 1/5W 0.5% -> FAE-RES:RS-0402-0R 1/5W 0.5%
- R150, R152, R155, R156, R157, R158, R159, R161, R162, R163, R168, R169: symbol Flatburn_V4_sym_library:RS-0402-100K 1/16W 1% -> FAE-RES:RS-0402-100K 1/16W 1%
- R151: symbol Flatburn_V4_sym_library:RS-0402-10K 1/16W 1% -> FAE-RES:RS-0402-10K 1/16W 1%
- R160: symbol Flatburn_V4_sym_library:RS-0402-2K2 1/16W 1% -> FAE-RES:RS-0402-2K2 1/16W 1%
- R164: symbol Flatburn_V4_sym_library:RS-0402-1K 1/16W 1% -> FAE-RES:RS-0402-1K 1/16W 1%
- TP21, TP22, TP23: symbol Flatburn_V4_sym_library:TestPoint -> Connector:TestPoint
- U10: symbol Flatburn_V4_sym_library:OPAMP - 5V/1MHz - AD8541ARTZ-REEL7 -> FAE-IC:OPAMP - 5V/1MHz - AD8541ARTZ-REEL7
- U11: symbol Flatburn_V4_sym_library:LEVEL SHIF - 2x - TXS0102DQER -> FAE-IC:LEVEL SHIF - 2x - TXS0102DQER
- U12: symbol Flatburn_V4_sym_library:RF AMPLIFIER GNSS- 1550-1615MHz/20dB - BGA725L6E6327FTSA1 -> FAE-IC:RF AMPLIFIER GNSS- 1550-1615MHz/20dB - BGA725L6E6327FTSA1
- U13: symbol Flatburn_V4_sym_library:SAW FILTER - GNSS/1575MHz - B39162B9416K610 -> FAE-SIGNAL:SAW FILTER - GNSS/1575MHz - B39162B9416K610
