File: hardware/electronics/mcu.kicad_sch (KiCad schematic)
At the start: 76 parts, among them J10 DM3CS-SF, J9 MDT420E01001, Q16 DMN63D8L-7, Q17 BSS209PWH6327XTSA1, U8 TPS3823-33DBVR, U9 TLC59711PWPR

Commit message: v5_update
Parts:
- ASS3: value NU -> B404x; symbol Flatburn_V4_sym_library:SOM - B404x -> FAE-MCU:SOM - B404x
- BUZ1: symbol Flatburn_V4_sym_library:BUZZER - 3V - ST-025BH -> FAE-BUZZ:BUZZER - 3V - ST-025BH
- C100, C103, C105: symbol Flatburn_V4_sym_library:CS-C-0603-10u/10V-10% -> FAE-CAP:CS-C-0603-10u/10V-10%
- C101, C102, C104, C93, C94, C95, C96, C99: symbol Flatburn_V4_sym_library:CS-C-0402-100n/50V-10% -> FAE-CAP:CS-C-0402-100n/50V-10%
- C97, C98: symbol Flatburn_V4_sym_library:CS-C-0402-33p/50V-5% -> FAE-CAP:CS-C-0402-33p/50V-5%
- D1: symbol Flatburn_V4_sym_library:DIODE - VR100V/0.15A - 1N4148WS -> FAE-DIODES:DIODE - VR100V/0.15A - 1N4148WS
- J10: symbol Flatburn_V4_sym_library:uSD - HIGED - DM3CS-SF -> FAE-CONN:uSD - HIGED - DM3CS-SF
- J9: symbol Flatburn_V4_sym_library:M2 - J-75-0050-MOS-M2-E - MDT420E01001 -> FAE-CONN:M2 - J-75-0050-MOS-M2-E - MDT420E01001
- L7: symbol Flatburn_V4_sym_library:FER - 220Ohm/2A - 25% - BLM21PG221SN1D -> FAE-IND:FER - 220Ohm/2A - 25% - BLM21PG221SN1D
- LD2, LD3: symbol Flatburn_V4_sym_library:LED - RGB - RIGHT ANGLE - 5mA -> FAE-DIODES:LED - RGB - RIGHT ANGLE - 5mA
- PB2, PB3: symbol Flatburn_V4_sym_library:PB - 1571634-2 - 24V 50mA -> FAE-SWITCH:PB - 1571634-2 - 24V 50mA
- Q16: symbol Flatburn_V4_sym_library:NMOS - 30V 350mA - DMN63D8L-7 -> FAE-TRANSISTOR:NMOS - 30V 350mA - DMN63D8L-7
- Q17: symbol Flatburn_V4_sym_library:PMOS - 20V 630mA - BSS209PWH6327XTSA1 -> FAE-TRANSISTOR:PMOS - 20V 630mA - BSS209PWH6327XTSA1
- R103, R104, R106, R109, R110, R111, R119, R120, R121, R122, R123, R126: symbol Flatburn_V4_sym_library:RS-0402-100K 1/16W 1% -> FAE-RES:RS-0402-100K 1/16W 1%
- R105, R128: symbol Flatburn_V4_sym_library:RS-0402-0R 1/5W 0.5% -> FAE-RES:RS-0402-0R 1/5W 0.5%
- R107, R108: value 2.2k -> 4.7k; symbol Flatburn_V4_sym_library:RS-0402-2K2 1/16W 1% -> FAE-RES:RS-0402-4K7 1/16W 1%; Distributor FAE-035095 -> FAE-025131
- R112, R113, R114, R125, R127: symbol Flatburn_V4_sym_library:RS-0402-100R 1/16W 1% -> FAE-RES:RS-0402-100R 1/16W 1%
- R115, R136, R225: symbol Flatburn_V4_sym_library:RS-0402-10K 1/16W 1% -> FAE-RES:RS-0402-10K 1/16W 1%
- R116, R117: symbol Flatburn_V4_sym_library:RS-0402-0R 100mW 0.1% -> FAE-RES:RS-0402-0R 100mW 0.1%
- R118: symbol Flatburn_V4_sym_library:RS-0402-470R 1/16W 1% -> FAE-RES:RS-0402-470R 1/16W 1%
- R124: symbol Flatburn_V4_sym_library:RS-0402-270R 1/16W 1% -> FAE-RES:RS-0402-270R 1/16W 1%
- R129, R130, R131, R132, R133, R134, R135: symbol Flatburn_V4_sym_library:RS-0402-47K 1/16W 1% -> FAE-RES:RS-0402-47K 1/16W 1%
- R137, R138, R139, R140, R141, R142, R143: symbol Flatburn_V4_sym_library:RS-0402-33R 1/16W 1% -> FAE-RES:RS-0402-33R 1/16W 1%
- R144: symbol Flatburn_V4_sym_library:RS-0402-9K88 1/16W 0.5% -> FAE-RES:RS-0402-9K88 1/16W 0.5%
- TP18, TP19, TP20: symbol Flatburn_V4_sym_library:TestPoint -> Connector:TestPoint
- TVS21, TVS22: symbol Flatburn_V4_sym_library:TVS/ESD - UNI - 5,5V/500W_1 - D5V0S1U2LP-7B -> FAE-PROT:TVS/ESD - UNI - 5,5V/500W_1 - D5V0S1U2LP-7B
- TVS23: symbol Flatburn_V4_sym_library:TVS/ESD IC - UNI- 5V/32W - D3V3F8U9LP3810-7 -> FAE-PROT:TVS/ESD IC - UNI- 5V/32W - D3V3F8U9LP3810-7
- U8: symbol Flatburn_V4_sym_library:SUPERVISOR - 5V - TPS3823-33DBVR -> FAE-IC:SUPERVISOR - 5V - TPS3823-33DBVR
- U9: symbol Flatburn_V4_sym_library:DRIVER LED - 18V/60mA - 16Bit/12Ch - TLC59711PWPR -> FAE-IC:DRIVER LED - 18V/60mA - 16Bit/12Ch - TLC59711PWPR
