File: hardware/electronics/power.kicad_sch (KiCad schematic)
At the start: 85 parts, among them J8 STRIP-2P-M, Q2 SISH402DN-T1-GE3, Q3 SISH402DN-T1-GE3, Q4 SISH402DN-T1-GE3, Q5 SISH402DN-T1-GE3, Q6 BSS84WQ-7-F, U1 TPS25730DREFR, U2 BQ25798RQMR

Commit message: v5_update
Parts:
- C10, C9: symbol Flatburn_V4_sym_library:CS-C-0402-330p/10V-10% -> FAE-CAP:CS-C-0402-330p/10V-10%
- C11, C8: symbol Flatburn_V4_sym_library:CS-C-0603-10u/10V-10% -> FAE-CAP:CS-C-0603-10u/10V-10%
- C12, C21: symbol Flatburn_V4_sym_library:CS-C-0603-4.7u/10V-10% -> FAE-CAP:CS-C-0603-4.7u/10V-10%
- C13: symbol Flatburn_V4_sym_library:CS-P-8x10-47u/50V-20% -> FAE-CAP:CS-P-8x10-47u/50V-20%
- C14, C5, C6: symbol Flatburn_V4_sym_library:CS-C-0402-10n/50V-10% -> FAE-CAP:CS-C-0402-10n/50V-10%
- C15, C16: symbol Flatburn_V4_sym_library:CS-C-0402-47n/25V-10% -> FAE-CAP:CS-C-0402-47n/25V-10%
- C17, C18, C24, C25, C26: symbol Flatburn_V4_sym_library:CS-C-0805-10u/50V-10% -> FAE-CAP:CS-C-0805-10u/50V-10%
- C19, C27, C33: symbol Flatburn_V4_sym_library:CS-C-0402-100n/50V-10% -> FAE-CAP:CS-C-0402-100n/50V-10%
- C20: symbol Flatburn_V4_sym_library:CS-C-0402-1n/50V-10% -> FAE-CAP:CS-C-0402-1n/50V-10%
- C22, C23: symbol Flatburn_V4_sym_library:CS-C-0603-10u/25V-20% -> FAE-CAP:CS-C-0603-10u/25V-20%
- C28, C29, C30, C31, C32: symbol Flatburn_V4_sym_library:CS-C-0603-10u/25V-10% -> FAE-CAP:CS-C-0603-10u/25V-10%
- C7: symbol Flatburn_V4_sym_library:CS-C-0603-4.7u/35V-10% -> FAE-CAP:CS-C-0603-4.7u/35V-10%
- DZ2, DZ3: symbol Flatburn_V4_sym_library:ZENER - UNI- 12V/300mW - BZT52C12T-7 -> FAE-DIODES:ZENER - UNI- 12V/300mW - BZT52C12T-7
- J8: symbol Flatburn_V4_sym_library:STRIP - 2P - MDT -> FAE-CONN:STRIP - 2P - MDT
- L3: symbol Flatburn_V4_sym_library:PW - 10uH/15.8A - SPM6550T-1R0M100A -> FAE-IND:PW - 10uH/15.8A - SPM6550T-1R0M100A
- LD1: symbol Flatburn_V4_sym_library:LED - RED - RIGHT ANGLE - 2.6V 20mA -> FAE-DIODES:LED - RED - RIGHT ANGLE - 2.6V 20mA
- PB1: symbol Flatburn_V4_sym_library:PB - 1571634-2 - 24V 50mA -> FAE-SWITCH:PB - 1571634-2 - 24V 50mA
- Q2, Q3, Q4, Q5: symbol Flatburn_V4_sym_library:NMOS - 30V 35A - SISH402DN-T1-GE3 -> FAE-TRANSISTOR:NMOS - 30V 35A - SISH402DN-T1-GE3
- Q6: symbol Flatburn_V4_sym_library:PMOS - 50V 130mA - BSS84WQ-7-F -> FAE-TRANSISTOR:PMOS - 50V 130mA - BSS84WQ-7-F
- R10, R11, R12, R13, R14, R15, R16, R17, R18, R19, R24, R29, R33, R6, R7, R8, R9: symbol Flatburn_V4_sym_library:RS-0402-10K 1/16W 1% -> FAE-RES:RS-0402-10K 1/16W 1%
- R20, R25: symbol Flatburn_V4_sym_library:RS-0603-294R 1/16W 1% -> FAE-RES:RS-0603-294R 1/16W 1%
- R21: symbol Flatburn_V4_sym_library:RS-0402-255K 1/16W 1% -> FAE-RES:RS-0402-255K 1/16W 1%
- R22: symbol Flatburn_V4_sym_library:RS-0402-100K 1/16W 1% -> FAE-RES:RS-0402-100K 1/16W 1%
- R23: symbol Flatburn_V4_sym_library:RS-0402-560R 1/16W 1% -> FAE-RES:RS-0402-560R 1/16W 1%
- R26: symbol Flatburn_V4_sym_library:RS-0603-0R 1/10W 2A -> FAE-RES:RS-0603-0R 1/10W 2A
- R27: symbol Flatburn_V4_sym_library:RS-0402-0R 1/5W 0.5% -> FAE-RES:RS-0402-0R 1/5W 0.5%
- R28, R31: symbol Flatburn_V4_sym_library:RS-0402-100R 1/16W 1% -> FAE-RES:RS-0402-100R 1/16W 1%
- R30: symbol Flatburn_V4_sym_library:RS-0402-5K23 1/16W 1% -> FAE-RES:RS-0402-5K23 1/16W 1%
- R32: symbol Flatburn_V4_sym_library:RS-0402-30K1 1/16W 1% -> FAE-RES:RS-0402-30K1 1/16W 1%
- R34: symbol Flatburn_V4_sym_library:RS-0603-6K04 1/16W 1% -> FAE-RES:RS-0603-6K04 1/16W 1%
- R35: symbol Flatburn_V4_sym_library:RS-0603-3K 1/16W 1% -> FAE-RES:RS-0603-3K 1/16W 1%
- R5: symbol Flatburn_V4_sym_library:RS-1206-0R 1/4W 3,5A -> FAE-RES:RS-1206-0R 1/4W 3,5A
- TP1, TP10, TP2, TP3, TP37, TP4, TP5, TP6, TP7, TP8, TP9: symbol Flatburn_V4_sym_library:TestPoint -> Connector:TestPoint
- TVS19: symbol Flatburn_V4_sym_library:TVS/ESD - UNI - 5,5V/500W_1 - D5V0S1U2LP-7B -> FAE-PROT:TVS/ESD - UNI - 5,5V/500W_1 - D5V0S1U2LP-7B
- U1: symbol Flatburn_V4_sym_library:USB - PD INTERFACE - TPS25730DREFR -> FAE-IC:USB - PD INTERFACE - TPS25730DREFR
- U2: symbol Flatburn_V4_sym_library:BAT-CHARGE - BQ25798RQMR -> FAE-PWR:BAT-CHARGE - BQ25798RQMR
