File: hardware/electronics/power2.kicad_sch (KiCad schematic)
At the start: 153 parts, among them Q10 SISS27DN-T1-GE3, Q11 SISS27DN-T1-GE3, Q12 DMN63D8L-7, Q13 DMN63D8L-7, Q14 DMN63D8L-7, Q15 DMN63D8L-7, Q7 SISS27DN-T1-GE3, Q8 SISS27DN-T1-GE3, Q9 SISS27DN-T1-GE3, SW1 R10307RN02Q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

Commit message: v5_update
Parts:
- C34, C35, C39, C40, C44, C48, C49, C50, C51, C52, C55, C60, C66, C71, C79, C81, C82, C83, C84, C85, C86, C87, C88: symbol Flatburn_V4_sym_library:CS-C-0402-100n/50V-10% -> FAE-CAP:CS-C-0402-100n/50V-10%
- C36: symbol Flatburn_V4_sym_library:CS-C-0402-10p/50V-5% -> FAE-CAP:CS-C-0402-10p/50V-5%
- C37, C38: symbol Flatburn_V4_sym_library:CS-EL-6.3x7.7-220u/25V-20% -> FAE-CAP:CS-EL-6.3x7.7-220u/25V-20%
- C41, C42, C43: symbol Flatburn_V4_sym_library:CS-C-0805-1u/50V-10% -> FAE-CAP:CS-C-0805-1u/50V-10%
- C45, C46, C47: symbol Flatburn_V4_sym_library:CS-C-0603-1u/25V-10% -> FAE-CAP:CS-C-0603-1u/25V-10%
- C53, C54, C56, C57, C64, C65, C67, C68, C76, C77: symbol Flatburn_V4_sym_library:CS-C-0603-10u/25V-10% -> FAE-CAP:CS-C-0603-10u/25V-10%
- C58: symbol Flatburn_V4_sym_library:CS-C-0603-330p/25V-5% -> FAE-CAP:CS-C-0603-330p/25V-5%
- C59: symbol Flatburn_V4_sym_library:CS-C-0603-22n/16V-5% -> FAE-CAP:CS-C-0603-22n/16V-5%
- C61, C62, C63, C72, C73, C74, C75: symbol Flatburn_V4_sym_library:CS-C-0805-22u/16V-20% -> FAE-CAP:CS-C-0805-22u/16V-20%
- C69: symbol Flatburn_V4_sym_library:CS-C-0603-560p/25V-5% -> FAE-CAP:CS-C-0603-560p/25V-5%
- C70: symbol Flatburn_V4_sym_library:CS-C-0603-27n/25V-5% -> FAE-CAP:CS-C-0603-27n/25V-5%
- C78: symbol Flatburn_V4_sym_library:CS-C-0402-3.3n/25V-10% -> FAE-CAP:CS-C-0402-3.3n/25V-10%
- C80: symbol Flatburn_V4_sym_library:CS-C-0603-22u/6.3V-20% -> FAE-CAP:CS-C-0603-22u/16V-20%; Distributor M-81-GRM188R60J226ME0D -> M-581-KGM15CR51C226MT; MPN GRM188R60J226MEA0D -> KGM15CR51C226MT; Price Distributor Cad 0,143 -> 0,404
- C89, C90, C91, C92: symbol Flatburn_V4_sym_library:CS-C-0603-10u/10V-10% -> FAE-CAP:CS-C-0603-10u/10V-10%
- L4, L5: symbol Flatburn_V4_sym_library:PW - 1uH/8.8A - XGL4020-102MEC -> FAE-IND:PW - 1uH/8.8A - XGL4020-102MEC
- L6: symbol Flatburn_V4_sym_library:PW - 2.2uH/6.3A -XGL4025-222MEC -> FAE-IND:PW - 2.2uH/6.3A -XGL4025-222MEC
- Q10, Q11, Q7, Q8, Q9: symbol Flatburn_V4_sym_library:PMOS - 30V 50A - SISS27DN-T1-GE3 -> FAE-TRANSISTOR:PMOS - 30V 50A - SISS27DN-T1-GE3
- Q12, Q13, Q14, Q15: symbol Flatburn_V4_sym_library:NMOS - 30V 350mA - DMN63D8L-7 -> FAE-TRANSISTOR:NMOS - 30V 350mA - DMN63D8L-7
- R100, R101, R102, R40, R41, R42, R43, R46, R47, R48, R54, R55, R56, R57, R62, R63, R64, R65, R70, R71, R72, R73, R99: symbol Flatburn_V4_sym_library:RS-0402-10K 1/16W 1% -> FAE-RES:RS-0402-10K 1/16W 1%
- R36, R37, R38, R39: symbol Flatburn_V4_sym_library:RS-1206-0R016 1/4W 1% -> FAE-RES:RS-1206-0R016 1/4W 1%
- R44, R45, R49, R50, R51, R52: symbol Flatburn_V4_sym_library:RS-0603-10R 1/10W 1% -> FAE-RES:RS-0603-10R 1/10W 1%
- R53, R95, R96, R97, R98: symbol Flatburn_V4_sym_library:RS-0402-100R 1/16W 1% -> FAE-RES:RS-0402-100R 1/16W 1%
- R58: symbol Flatburn_V4_sym_library:RS-0603-50m 1/2W 1% -> FAE-RES:RS-0603-50m 1/2W 1%
- R59: symbol Flatburn_V4_sym_library:RS-0603-20m 1/2W 1% -> FAE-RES:RS-0603-20m 1/2W 1%
- R60, R61, R78, R83, R84, R85, R86: symbol Flatburn_V4_sym_library:RS-0402-100K 1/16W 1% -> FAE-RES:RS-0402-100K 1/16W 1%
- R66: symbol Flatburn_V4_sym_library:RS-0402-43K 1/16W 1% -> FAE-RES:RS-0402-43K 1/16W 1%
- R67: symbol Flatburn_V4_sym_library:RS-0402-31K2 1/16W 0.5% -> FAE-RES:RS-0402-31K2 1/16W 0.5%
- R68: symbol Flatburn_V4_sym_library:RS-0603-6K34 1/16W 0.5% -> FAE-RES:RS-0603-6K34 1/16W 0.5%
- R69: symbol Flatburn_V4_sym_library:RS-0603-5K23 1/16W 1% -> FAE-RES:RS-0603-5K23 1/16W 1%
- R74, R76, R87, R89, R91, R93: symbol Flatburn_V4_sym_library:RS-0402-0R 1/5W 0.5% -> FAE-RES:RS-0402-0R 1/5W 0.5%
- R75, R77: symbol Flatburn_V4_sym_library:RS-0402-9K31 1/16W 1% -> FAE-RES:RS-0402-9K31 1/16W 1%
- R79, R80, R81, R82: symbol Flatburn_V4_sym_library:RS-1206-0R 1/4W 3,5A -> FAE-RES:RS-1206-0R 1/4W 3,5A
- R88, R90, R92, R94: symbol Flatburn_V4_sym_library:RS-0402-12K 1/16W 1% -> FAE-RES:RS-0402-12K 1/16W 1%
- SW1: symbol Flatburn_V4_sym_library:SW - ROTARY 3P - FS22ABP - 125V 5A -> FAE-SWITCH:SW - ROTARY 3P - FS22ABP - 125V 5A
- SW2: symbol Flatburn_V4_sym_library:SW - DPDT - FS22ABP - 28V 1A -> FAE-SWITCH:SW - DPDT - FS22ABP - 28V 1A
- TP11, TP12, TP13, TP14, TP15, TP16, TP17: symbol Flatburn_V4_sym_library:TestPoint -> Connector:TestPoint
- TVS20: symbol Flatburn_V4_sym_library:TVS/ESD - UNI- 10V/200W - SMF10A-E3-08 -> FAE-PROT:TVS/ESD - UNI- 10V/200W - SMF10A-E3-08
- U3, U4: symbol Flatburn_V4_sym_library:CURRENT SENSE - 700uA - ISL28022FUZ -> FAE-IC:CURRENT SENSE - 700uA - ISL28022FUZ
- U5, U6: symbol Flatburn_V4_sym_library:BUCK-BOOST - 3-36Vin - 0.8-22Vout - 4A -TPS552872RYQR -> FAE-PWR:BUCK-BOOST - 3-36Vin - 0.8-22Vout - 4A -TPS552872RYQR
- U7: symbol Flatburn_V4_sym_library:BUCK - 3-17Vin - 3.3Vout - 2A - TPS62142 -> FAE-PWR:BUCK - 3-17Vin - 3.3Vout - 2A - TPS62142
