File: hardware/electronics/sensors.kicad_sch (KiCad schematic)
At the start: 76 parts, among them Q18 DMN63D8L-7, U14 74LV4066PW, U15 BME280, U16 KXTJ3-1057, U17 AD8541ARTZ, U18 TXS0102DQER, U19 MCP6022-I/SN, U20 LTC1966IMS8, U21 CMM-2718AT-42316-TR, U22 MCP6022-I/SN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

Commit message: v5_update
Parts:
- C122, C123, C124, C125, C126, C128, C129, C130, C131, C133, C134, C135, C136, C138, C140, C141, C142, C143, C145: symbol Flatburn_V4_sym_library:CS-C-0402-100n/50V-10% -> FAE-CAP:CS-C-0402-100n/50V-10%
- C127, C132, C137, C139, C144: symbol Flatburn_V4_sym_library:CS-C-0402-1u/16V-10% -> FAE-CAP:CS-C-0402-1u/16V-10%
- C146: symbol Flatburn_V4_sym_library:CS-C-0603-10u/10V-10% -> FAE-CAP:CS-C-0603-10u/10V-10%
- Q18: symbol Flatburn_V4_sym_library:NMOS - 30V 350mA - DMN63D8L-7 -> FAE-TRANSISTOR:NMOS - 30V 350mA - DMN63D8L-7
- R170, R175, R176, R181, R185, R188, R190, R194: symbol Flatburn_V4_sym_library:RS-0402-100K 1/16W 1% -> FAE-RES:RS-0402-100K 1/16W 1%
- R171, R177, R179: symbol Flatburn_V4_sym_library:RS-0402-0R 1/5W 0.5% -> FAE-RES:RS-0402-0R 1/5W 0.5%
- R172, R173, R178, R180, R182, R192, R193, R196, R197, R200, R201, R202: symbol Flatburn_V4_sym_library:RS-0402-10K 1/16W 1% -> FAE-RES:RS-0402-10K 1/16W 1%
- R174: symbol Flatburn_V4_sym_library:RS-0402-4K7 1/16W 1% -> FAE-RES:RS-0402-4K7 1/16W 1%
- R183, R184: value 2.2k -> 4.7k; symbol Flatburn_V4_sym_library:RS-0402-2K2 1/16W 1% -> FAE-RES:RS-0402-4K7 1/16W 1%; Distributor FAE-035095 -> FAE-025131
- R186, R187: symbol Flatburn_V4_sym_library:RS-0402-120K 1/16W 1% -> FAE-RES:RS-0402-120K 1/16W 1%
- R189, R195: symbol Flatburn_V4_sym_library:RS-0402-1M 1/16W 1% -> FAE-RES:RS-0402-1M 1/16W 1%
- R191: symbol Flatburn_V4_sym_library:RS-0603-390R 1/16W 1% -> FAE-RES:RS-0603-390R 1/16W 1%
- R198: symbol Flatburn_V4_sym_library:RS-0402-2K2 1/16W 1% -> FAE-RES:RS-0402-2K2 1/16W 1%
- R199: symbol Flatburn_V4_sym_library:RS-0402-1K 1/16W 1% -> FAE-RES:RS-0402-1K 1/16W 1%
- R203: symbol Flatburn_V4_sym_library:RS-0402-100R 1/16W 1% -> FAE-RES:RS-0402-100R 1/16W 1%
- TP24, TP25, TP26, TP27, TP28, TP29: symbol Flatburn_V4_sym_library:TestPoint -> Connector:TestPoint
- U14: symbol Flatburn_V4_sym_library:SWITCH - 4x - 74LV4066PW -> FAE-IC:SWITCH - 4x - 74LV4066PW
- U15: symbol Flatburn_V4_sym_library:HUM/TEMP/PRESS - BME280 -> FAE-SENS:HUM/TEMP/PRESS - BME280
- U16: symbol Flatburn_V4_sym_library:ACCEL- KXTJ3-1057 -> FAE-SENS:ACCEL- KXTJ3-1057
- U17: symbol Flatburn_V4_sym_library:OPAMP - 5V/1MHz - AD8541ARTZ-REEL7 -> FAE-IC:OPAMP - 5V/1MHz - AD8541ARTZ-REEL7
- U18: symbol Flatburn_V4_sym_library:LEVEL SHIF - 2x - TXS0102DQER -> FAE-IC:LEVEL SHIF - 2x - TXS0102DQER
- U19, U22: symbol Flatburn_V4_sym_library:OPAMP - 5.5V/10MHz - MCP6022-I/SN -> FAE-IC:OPAMP - 5.5V/10MHz - MCP6022-I/SN
- U20: symbol Flatburn_V4_sym_library:RMS-DC CONV - +-5.5V - TXS0102DQER_1 -> FAE-IC:RMS-DC CONV - +-5.5V - TXS0102DQER_1
- U21: symbol Flatburn_V4_sym_library:MIC - 94dB/1KHz - CMM-2718AT-42316-TR -> FAE-SENS:MIC - 94dB/1KHz - CMM-2718AT-42316-TR
- U23: symbol Flatburn_V4_sym_library:DAC - 12bit/2.7-5V - TXS0102DQER_1_1 -> FAE-IC:DAC - 12bit/2.7-5V - TXS0102DQER_1_1
