File: hardware/electronics/sensors2.kicad_sch (KiCad schematic)
At the start: 88 parts, among them U24 AD8541ARTZ, U25 AD8541ARTZ, U26 AD8541ARTZ, U27 TXS0102DQER, U28 TXS0102DQER, U29 TXS0102DQER, U30 TXS0102DQER, U31 MCP6022-I/SN, U32 REF5025AIDR, U33 ADS1256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

Commit message: v5_update
Parts:
- C147, C148, C149, C150, C151, C152, C153, C154, C155, C156, C157, C158, C159, C160, C162, C167, C168, C172, C174: symbol Flatburn_V4_sym_library:CS-C-0402-100n/50V-10% -> FAE-CAP:CS-C-0402-100n/50V-10%
- C161, C166, C171, C173: symbol Flatburn_V4_sym_library:CS-C-0402-1u/16V-10% -> FAE-CAP:CS-C-0402-1u/16V-10%
- C163: symbol Flatburn_V4_sym_library:CS-C-0603-4.7u/10V-10% -> FAE-CAP:CS-C-0603-4.7u/10V-10%
- C164: symbol Flatburn_V4_sym_library:CS-C-0603-1u/25V-10% -> FAE-CAP:CS-C-0603-1u/25V-10%
- C165: symbol Flatburn_V4_sym_library:CS-C-0603-22u/6.3V-20% -> FAE-CAP:CS-C-0603-22u/16V-20%; Distributor M-81-GRM188R60J226ME0D -> M-581-KGM15CR51C226MT; MPN GRM188R60J226MEA0D -> KGM15CR51C226MT; Price Distributor Cad 0,143 -> 0,404
- C169, C170: symbol Flatburn_V4_sym_library:CS-C-0603-18p/50V-5% -> FAE-CAP:CS-C-0603-18p/50V-5%
- L16: symbol Flatburn_V4_sym_library:PW - 2.2uH/0.35A -LQM18PN2R2MGHD -> FAE-IND:PW - 2.2uH/0.35A -LQM18PN2R2MGHD
- R204, R205, R206: symbol Flatburn_V4_sym_library:RS-0402-4K7 1/16W 1% -> FAE-RES:RS-0402-4K7 1/16W 1%
- R207, R208, R209: symbol Flatburn_V4_sym_library:RS-0402-0R 1/5W 0.5% -> FAE-RES:RS-0402-0R 1/5W 0.5%
- R210, R212, R214, R220, R221, R222, R223, R224, R239, R240, R241, R242: symbol Flatburn_V4_sym_library:RS-0402-100K 1/16W 1% -> FAE-RES:RS-0402-100K 1/16W 1%
- R211, R213, R215, R233, R234, R235, R236, R237, R238: symbol Flatburn_V4_sym_library:RS-0402-10K 1/16W 1% -> FAE-RES:RS-0402-10K 1/16W 1%
- R216, R217, R218, R219: value 2.2k -> 4.7k; symbol Flatburn_V4_sym_library:RS-0402-2K2 1/16W 1% -> FAE-RES:RS-0402-4K7 1/16W 1%; Distributor FAE-035095 -> FAE-025131
- R226, R228, R229, R230, R231, R232: symbol Flatburn_V4_sym_library:RS-0402-10R 1/16W 0.5% -> FAE-RES:RS-0402-10R 1/16W 0.5%
- R243, R244, R245: symbol Flatburn_V4_sym_library:RS-0402-100R 1/16W 1% -> FAE-RES:RS-0402-100R 1/16W 1%
- TP30, TP31, TP32, TP33, TP34, TP35: symbol Flatburn_V4_sym_library:TestPoint -> Connector:TestPoint
- U24, U25, U26: symbol Flatburn_V4_sym_library:OPAMP - 5V/1MHz - AD8541ARTZ-REEL7 -> FAE-IC:OPAMP - 5V/1MHz - AD8541ARTZ-REEL7
- U27, U28, U29, U30: symbol Flatburn_V4_sym_library:LEVEL SHIF - 2x - TXS0102DQER -> FAE-IC:LEVEL SHIF - 2x - TXS0102DQER
- U31, U34, U35: symbol Flatburn_V4_sym_library:OPAMP - 5.5V/10MHz - MCP6022-I/SN -> FAE-IC:OPAMP - 5.5V/10MHz - MCP6022-I/SN
- U32: symbol Flatburn_V4_sym_library:REF - 2.5V/10mA - REF5025AIDR -> FAE-IC:REF - 2.5V/10mA - REF5025AIDR
- U33: symbol Flatburn_V4_sym_library:ADC - 24Bit/8Ch - ADS1256IDBR -> FAE-IC:ADC - 24Bit/8Ch - ADS1256IDBR
- Y1: symbol Flatburn_V4_sym_library:CRYSTAL - 7.68MHz - HCM497680000ABJT -> FAE-XTAL:CRYSTAL - 7.68MHz - HCM497680000ABJT
Connections:
- net 5V_I2C_SCL: now also R218.2, U30.7 (B1); no longer R219.2, U30.6 (B2)
- net 5V_I2C_SDA: now also R219.2, U30.6 (B2); no longer R218.2, U30.7 (B1)
- net I2C_SCL: now also U30.2 (A1); no longer U30.3 (A2)
- net I2C_SDA: now also U30.3 (A2); no longer U30.2 (A1)
